File: rDuino.kicad_pcb (KiCad board)
At the start: 2 copper layers, 100.3 x 55.2 mm, 17 parts, among them J1 12v, P1 Switch, P2 GPS, P3 Joystick, P4 RTC-4pin, P5 Blue-tooth, P6 DHT22, P9 SPEAKER

Commit message: spk update
Parts:
- removed P9: SPEAKER, Connector_PinHeader_2.54mm:PinHeader_1x02_P2.54mm_Vertical
- added J2: Speaker, Connector_PinHeader_2.54mm:PinHeader_1x03_P2.54mm_Vertical, F.Cu at (142.9, 94.6)
Routing:
- net GND: track 374.3 -> 321.0 mm
- net Net-(A2-Pad12): track 26.5 -> 10.3 mm
- net Net-(J2-Pad2): track 22.3 -> 26.2 mm
- net +3V3: track 230.8 -> 233.7 mm
- added copper zone on F.Cu, net (none)
Other:
- board text added: "SPK"
